File: Test Rocket Board/Test Rocket Board.kicad_pcb (KiCad board)
At the start: 2 copper layers, 68 x 66 mm, 90 parts, among them IC1 ESP32-S3-WROOM-1U-N16, J1 Conn_01x03_Pin, J2 Conn_01x04_Pin, J3 USB_C_Receptacle_USB2.0_16P, J4 Conn_01x06_Socket, J5 Conn_01x02, J6 Conn_01x02_Socket, J7 Conn_01x05_Socket, J8 Conn_01x04_Pin, SW1 SW_Push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

Commit message: idk what this is
Other:
- board text added: "Test Board! RevB"
- board text removed: "Test Board! Rev 1"
Changed lines of the file:
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@@
 		)
 	)
-	(gr_text "Test Board!\nRev 1"
+	(gr_text "Test Board!\nRevB"
 		(at 173 78 0)
 		(layer "F.SilkS")
